Commit message: add humanoid
Signed-off-by: Nazwa Najmuddin <naznajmuddin@gmail.com>

File: description/robot_core.xacro (robot description, xacro)
@@ -25,14 +25,14 @@
     <link name="chassis">
         <visual>
+            <origin xyz = "0.15 0 0.055" />
+            <geometry>
+                <box size="0.3 0.3 0.05" />
+            </geometry>
+            <material name="white"/>
+        </visual>
+        <collision>
             <origin xyz = "0.15 0 0.075" />
             <geometry>
-                <box size="0.3 0.3 0.15" />
-            </geometry>
-            <material name="white"/>
-        </visual>
-        <collision>
-            <origin xyz = "0.15 0 0.075" />
-            <geometry>
-                <box size="0.3 0.3 0.15" />
+                <box size="0.3 0.3 0.05" />
             </geometry>
         </collision>
@@ -42,5 +42,5 @@
     </link>
     <gazebo reference="chassis">
-        <material>Gazebo/White</material>
+        <material>Gazebo/Grey</material>
     </gazebo>
     <!-- LEFT WHEEL LINK -->
@@ -125,3 +125,113 @@
         <mu2 value="0.001" />
     </gazebo>
+    <!-- LEG LINK 1 -->
+    <joint name="leg1_joint" type="fixed">
+        <parent link="chassis"/>
+        <child link="leg1"/>
+        <origin xyz="0.15 0.1 0.25"/>
+    </joint>
+    <link name="leg1">
+        <visual>
+            <origin xyz="0 0 0"/>
+            <geometry>
+                <cylinder radius="0.05" length="0.4"/>
+            </geometry>
+            <material name="orange"/>
+        </visual>
+        <collision>
+            <origin xyz="0 0 0"/>
+            <geometry>
+                <cylinder radius="0.05" length="0.4"/>
+            </geometry>
+        </collision>
+        <xacro:inertial_cylinder mass="0.05" length="0.4" radius="0.05">
+            <origin xyz="0 0 0" rpy="0 0 0"/>
+        </xacro:inertial_cylinder>
+    </link>
+    <gazebo reference="leg1">
+        <material>Gazebo/Orange</material>
+    </gazebo>
+    <!-- LEG LINK 2 -->
+    <joint name="leg2_joint" type="fixed">
+        <parent link="chassis"/>
+        <child link="leg2"/>
+        <origin xyz="0.15 -0.1 0.25"/>
+    </joint>
+    <link name="leg2">
+        <visual>
+            <origin xyz="0 0 0"/>
+            <geometry>
+                <cylinder radius="0.05" length="0.4"/>
+            </geometry>
+            <material name="orange"/>
+        </visual>
+        <collision>
+            <origin xyz="0 0 0"/>
+            <geometry>
+                <cylinder radius="0.05" length="0.4"/>
+            </geometry>
+        </collision>
+        <xacro:inertial_cylinder mass="0.05" length="0.4" radius="0.05">
+            <origin xyz="0 0 0" rpy="0 0 0"/>
+        </xacro:inertial_cylinder>
+    </link>
+    <gazebo reference="leg2">
+        <material>Gazebo/Orange</material>
+    </gazebo>
+    <!-- UPPER BODY LINK -->
+    <joint name="upper_body_joint" type="fixed">
+        <parent link="base_link"/>
+        <child link="upper_body"/>
+        <origin xyz="0.05 0 0.55"/>
+    </joint>
+    <link name="upper_body">
+        <visual>
+            <origin xyz="0 0 0"/>
+            <geometry>
+                <box size="0.1 0.3 0.35"/>
+            </geometry>
+            <material name="white"/>
+        </visual>
+        <collision>
+            <origin xyz="0 0 0"/>
+            <geometry>
+                <box size="0.1 0.3 0.35"/>
+            </geometry>
+        </collision>
+        <xacro:inertial_box mass="0.1" x="0.2" y="0.2" z="0.2">
+            <origin xyz="0 0 0" rpy="0 0 0"/>
+        </xacro:inertial_box>
+    </link>
+    <gazebo reference="upper_body">
+        <material>Gazebo/White</material>
+    </gazebo>
+    <!-- HEAD LINK -->
+    <joint name="head_joint" type="fixed">
+        <parent link="upper_body"/>
+        <child link="head"/>
+        <origin xyz="0 0 0.25"/>
+        <!-- Adjust the XYZ values as needed -->
+    </joint>
+    <link name="head">
+        <visual>
+            <origin xyz="0 0 0"/>
+            <geometry>
+                <sphere radius="0.075"/>
+                <!-- Adjust the radius as needed -->
+            </geometry>
+            <material name="blue"/>
+        </visual>
+        <collision>
+            <origin xyz="0 0 0"/>
+            <geometry>
+                <sphere radius="0.075"/>
+            </geometry>
+        </collision>
+        <xacro:inertial_sphere mass="0.05" radius="0.1">
+            <origin xyz="0 0 0" rpy="0 0 0"/>
+        </xacro:inertial_sphere>
+    </link>
+    <gazebo reference="head">
+        <material>Gazebo/Blue</material>
+    </gazebo>
 </robot>

Commit message: add hands and joint state publisher
Signed-off-by: Nazwa Najmuddin <naznajmuddin@gmail.com>

File: description/robot_core.xacro (robot description, xacro)
@@ -204,5 +204,5 @@
     </link>
     <gazebo reference="upper_body">
-        <material>Gazebo/White</material>
+        <material>Gazebo/Black</material>
     </gazebo>
     <!-- HEAD LINK -->
@@ -233,5 +233,67 @@
     </link>
     <gazebo reference="head">
-        <material>Gazebo/Blue</material>
+        <material>Gazebo/White</material>
+    </gazebo>
+    <!-- HAND JOINT -->
+    <joint name="hand_joint" type="revolute">
+        <parent link="upper_body"/>
+        <child link="hand"/>
+        <origin xyz="0.0 -0.175 0.15"/>
+        <axis xyz="0 1 0"/>
+        <limit effort="100.0" velocity="0.5" lower="-3.1416" upper="3.1416"/>
+        <dynamics damping="0.1"/>
+    </joint>
+    <!-- HAND LINK -->
+    <link name="hand">
+        <visual>
+            <origin xyz="0.05 0 0"/>
+            <geometry>
+                <box size="0.2 0.05 0.05"/>
+            </geometry>
+            <material name="black"/>
+        </visual>
+        <collision>
+            <origin xyz="0.05 0 0"/>
+            <geometry>
+                <box size="0.2 0.05 0.05"/>
+            </geometry>
+        </collision>
+        <xacro:inertial_box mass="0.02" x="0.2" y="0.05" z="0.05">
+            <origin xyz="0 0 0" rpy="0 0 0"/>
+        </xacro:inertial_box>
+    </link>
+    <gazebo reference="hand">
+        <material>Gazebo/White</material>
+    </gazebo>
+    <!-- OPPOSITE HAND JOINT -->
+    <joint name="opposite_hand_joint" type="revolute">
+        <parent link="upper_body"/>
+        <child link="opposite_hand"/>
+        <origin xyz="0.0 0.175 0.15"/>
+        <axis xyz="0 1 0"/>
+        <limit effort="100.0" velocity="0.5" lower="-3.1416" upper="3.1416"/>
+        <dynamics damping="0.1"/>
+    </joint>
+    <!-- OPPOSITE HAND LINK -->
+    <link name="opposite_hand">
+        <visual>
+            <origin xyz="0.05 0 0"/>
+            <geometry>
+                <box size="0.2 0.05 0.05"/>
+            </geometry>
+            <material name="black"/>
+        </visual>
+        <collision>
+            <origin xyz="0.05 0 0"/>
+            <geometry>
+                <box size="0.2 0.05 0.05"/>
+            </geometry>
+        </collision>
+        <xacro:inertial_box mass="0.02" x="0.2" y="0.05" z="0.05">
+            <origin xyz="0 0 0" rpy="0 0 0"/>
+        </xacro:inertial_box>
+    </link>
+    <gazebo reference="opposite_hand">
+        <material>Gazebo/White</material>
     </gazebo>
 </robot>
