Commit message: add camera feature
Signed-off-by: Nazwa Najmuddin <naznajmuddin@gmail.com>

File: description/gazebo_control.xacro (robot description, xacro)
@@ -19,3 +19,33 @@
         </plugin>
     </gazebo>
+    <!-- GAZEBO CAMERA PLUGIN -->
+    <gazebo reference="camera">
+        <material>Gazebo/Yellow</material>
+        <sensor type="camera" name="my_camera">
+            <update_rate>20</update_rate>
+            <visualize>true</visualize>
+            <camera name="cam">
+                <horizontal_fov>1.3962634</horizontal_fov>
+                <image>
+                    <width>640</width>
+                    <height>480</height>
+                    <format>R8B8G8</format>
+                </image>
+                <clip>
+                    <near>0.02</near>
+                    <far>300</far>
+                </clip>
+                <noise>
+                    <type>gaussian</type>
+                    <mean>0.0</mean>
+                    <stddev>0.007</stddev>
+                </noise>
+            </camera>
+            <plugin name="camera_controller" filename="libgazebo_ros_camera.so">
+                <frame_name>camera_link_optical</frame_name>
+                <min_depth>0.1</min_depth>
+                <max_depth>500</max_depth>
+            </plugin>
+        </sensor>
+    </gazebo>
 </robot>

File: description/robot_core.xacro (robot description, xacro)
@@ -13,4 +13,7 @@
     <material name="black">
         <color rgba="0 0 0 1"/>
+    </material>
+    <material name="yellow">
+        <color rgba="1 1 0 1"/>
     </material>
     <!-- BASE LINK -->
@@ -191,5 +194,5 @@
                 <box size="0.1 0.3 0.35"/>
             </geometry>
-            <material name="white"/>
+            <material name="black"/>
         </visual>
         <collision>
@@ -211,5 +214,4 @@
         <child link="head"/>
         <origin xyz="0 0 0.25"/>
-        <!-- Adjust the XYZ values as needed -->
     </joint>
     <link name="head">
@@ -218,7 +220,6 @@
             <geometry>
                 <sphere radius="0.075"/>
-                <!-- Adjust the radius as needed -->
-            </geometry>
-            <material name="blue"/>
+            </geometry>
+            <material name="white"/>
         </visual>
         <collision>
@@ -251,5 +252,5 @@
                 <box size="0.2 0.05 0.05"/>
             </geometry>
-            <material name="black"/>
+            <material name="white"/>
         </visual>
         <collision>
@@ -282,5 +283,5 @@
                 <box size="0.2 0.05 0.05"/>
             </geometry>
-            <material name="black"/>
+            <material name="white"/>
         </visual>
         <collision>
@@ -297,3 +298,28 @@
         <material>Gazebo/White</material>
     </gazebo>
+    <!-- CAMERA JOINT -->
+    <joint name="camera_joint" type="fixed">
+        <parent link="head"/>
+        <child link="camera"/>
+        <origin xyz="0 0 0.1"/>
+    </joint>
+    <!-- CAMERA LINK -->
+    <link name="camera">
+        <visual>
+            <origin xyz="0 0 0"/>
+            <geometry>
+                <box size="0.05 0.05 0.05"/>
+            </geometry>
+            <material name="yellow"/>
+        </visual>
+        <collision>
+            <origin xyz="0 0 0"/>
+            <geometry>
+                <box size="0.05 0.05 0.05"/>
+            </geometry>
+        </collision>
+        <xacro:inertial_box mass="0.02" x="0.1" y="0.1" z="0.1">
+            <origin xyz="0 0 0" rpy="0 0 0"/>
+        </xacro:inertial_box>
+    </link>
 </robot>
